Commit message: added floor to room

File: src/environment/room.urdf (robot description, URDF)
Before this commit: robot room, 2 links, 1 joints
Links:
- link walls: geometry collision box size=0.1 10.0 10.0; collision box size=0.1 10.0 10.0

Commit message: added floor to the urdf

File: src/environment/room.urdf (robot description, URDF)
Before this commit: robot room, 2 links, 1 joints
Links:
- added link floor, mass 0.0; collision box size=10.0 10.0 0.1; visual box size=10.0 10.0 0.1
Joints:
- added joint world_to_floor: type fixed, parent world, child floor
