Commit message: Change table to cylinder shape (radius 0.5, height 0.625)

File: src/environment/table.urdf (robot description, URDF)
Before this commit: robot table, 6 links, 5 joints
Links:
- removed link leg1
- removed link leg2
- removed link leg3
- removed link leg4
- removed link table_base
- removed link table_top
- added link table_cylinder, mass 15.0; collision cylinder length=0.625 radius=0.5; visual cylinder length=0.625 radius=0.5
Joints:
- removed joint base_to_top
- removed joint j1
- removed joint j2
- removed joint j3
- removed joint j4
