Commit message: updated cognitive to include sensor module

File: src/robot/robot.urdf (robot description, URDF)
Before this commit: robot iis_robot, 17 links, 16 joints
Links:
- added link lidar_link
Joints:
- added joint lidar_joint: type fixed, parent base_link, child lidar_link, origin xyz=0 0 0.18 rpy=0 0 0

Commit message: Fix robot grasping: IK mapping, table approach standoff, rear avoidance, keep-out zone
Major improvements to navigate-to-grasp mission:

Core fixes:
- Fixed IK index mapping in motion_control.py: properly map arm joint indices to IK solution values
- Increased grasp timeout from 5s to 8s for multi-phase sequence (fsm.py)
- Increased standoff distance to 1.1m to keep robot clear of table footprint
- Added virtual table keep-out zone with elliptical distance calculation

Approach strategy:
- NAVIGATE and APPROACH states now route to standoff position, not directly at cylinder
- Standoff computed perpendicular to table's long side (1.5m edge) using table orientation
- Orbit mode: robot orbits table at 2m radius when close but target not yet found
- Path planner increased obstacle clearance from 0.5m to 1.0m for larger table footprint

Obstacle avoidance:
- Added rear obstacle detection to prevent backing into walls
- Virtual keep-out zone (0.6m normal / 0.2m approach mode) prevents driving under table
- Lidar-blind table detected via geometric calculation from initial map
- Relaxed avoidance thresholds during approach phase

Multi-phase grasp:
- Phase 1 (0-2.5s): Open gripper, raise lift, IK to position above target
- Phase 2 (2.5-5.5s): Lower arm to grasp position with gripper open
- Phase 3 (5.5-8s): Close gripper on cylinder

Failure recovery:
- On grasp failure, robot backs away with rear obstacle avoidance
- Stow arm joints and lower lift during backup
- Open gripper to release partial grasps
- Reset standoff/waypoint for fresh approach on retry

File: src/robot/robot.urdf (robot description, URDF)
Before this commit: robot iis_robot, 17 links, 16 joints
Links:
- link base_link: mass 20.0 -> 5.0
- link torso_link: mass 10.0 -> 2.0
Joints:
- joint arm_base_joint: limit lower=-3.14 upper=0 effort=10.0 velocity=1.0 -> lower=0 upper=3.14 effort=10.0 velocity=1.0
- joint bl_wheel_joint: axis 0 0 1 -> 0 0 -1
- joint br_wheel_joint: axis 0 0 1 -> 0 0 -1
- joint fl_wheel_joint: axis 0 0 1 -> 0 0 -1
- joint fr_wheel_joint: axis 0 0 1 -> 0 0 -1
- joint lift_joint: origin xyz=0 -0.1 -0.15 rpy=0 0 0 -> xyz=0 0.1 -0.15 rpy=0 0 0

Commit message: first try without learning to fix robot

File: src/robot/robot.urdf (robot description, URDF)
Before this commit: robot iis_robot, 21 links, 20 joints
Links:
- removed link elbow_link_start
- link base_link: mass 5.0 -> 12.0
Joints:
- removed joint elbow_joint_start
- joint camera_joint: origin xyz=0.25 0 0.15 rpy=0 0 0 -> xyz=0.25 0 0.45 rpy=0 0 0
- joint elbow_joint: axis 0 1 0 -> 1 0 0
- joint shoulder_joint: axis 0 1 0 -> 1 0 0
- joint wrist_joint_start: origin (none) -> xyz=0 0 0 rpy=0 0 0
- joint wrist_pitch_joint: axis 0 1 0 -> 1 0 0
- joint wrist_roll_joint: parent wrist_pitch_link -> wrist_link_start
- joint wrist_roll_joint_cup: origin xyz=0 0 0.03 -> xyz=0 0 0 rpy=0 0 0; parent wrist_pitch_link -> wrist_roll_link

Commit message: changed camera position + added more obstacles

File: src/robot/robot.urdf (robot description, URDF)
Before this commit: robot iis_robot, 17 links, 16 joints
Joints:
- joint camera_joint: origin xyz=0.25 0 0.15 rpy=0 0 0 -> xyz=0.0 0.0 0.06 rpy=0 0.2 0; parent base_link -> gripper_base

Commit message: updated cognitive and robot

File: src/robot/robot.urdf (robot description, URDF)
Before this commit: robot iis_robot, 18 links, 17 joints
Links:
- link torso_link: mass 10.0 -> 4.0; geometry collision cylinder length=0.4 radius=0.05; visual box size=0.3 0.3 0.6

Commit message: Fix 12 bugs from comprehensive code review
Critical fixes:
- sensor_preprocessing.py: Remove GaussianBlur on normalized depth buffer
  (corrupts nonlinear depth values before meter conversion)
- world_builder.py: Apply rotated dx/dy offset to target position on table
  (target was always placed at table center, ignoring computed offset)
- world_builder.py: Use __file__-relative paths for URDF loading
  (portable execution from any working directory)

Collision/navigation fixes:
- action_planning.py: Increase obstacle clearance from 1.0m to 1.5m
  (accounts for 0.4m obstacle cubes + 0.5m robot width)
- action_planning.py: Increase waypoint offset from 1.0m to 1.5m
- cognitive_architecture.py: Fix lidar ray indices for left/right detection
  (left: rays 5-12 centered on 90deg, right: rays 24-31 centered on 270deg)
- cognitive_architecture.py: Add emergency braking during close approach
  (hard-stop if front obstacle < 0.15m when lidar avoidance disabled)

Grasping fixes:
- robot.urdf: Expand joint limits for arm reachability
  (arm_base: [-pi,pi], shoulder: [-1.0,1.57], elbow: [-0.5,2.0])
- fsm.py: Increase grasp timeout from 8s to 20s (IK convergence needs time)
- cognitive_architecture.py: Replace unreliable motor torque contact detection
  with p.getContactPoints (simulates touch sensor on gripper)

Other fixes:
- cognitive_architecture.py: Increase min_area from 10 to 50 (noise filter)
- cognitive_architecture.py: Add loop termination after SUCCESS holds 3s

File: src/robot/robot.urdf (robot description, URDF)
Before this commit: robot iis_robot, 21 links, 20 joints
Joints:
- joint arm_base_joint: limit lower=0 upper=3.14 effort=10.0 velocity=1.0 -> lower=-3.14 upper=3.14 effort=10.0 velocity=1.0
- joint elbow_joint: limit lower=0.0 upper=2.0 effort=10.0 velocity=1.0 -> lower=-0.5 upper=2.0 effort=10.0 velocity=1.0
- joint shoulder_joint: limit lower=0.0 upper=1.57 effort=10.0 velocity=1.0 -> lower=-1.0 upper=1.57 effort=10.0 velocity=1.0

Commit message: adjusted camera and base mass

File: src/robot/robot.urdf (robot description, URDF)
Before this commit: robot iis_robot, 17 links, 16 joints
Links:
- added link elbow_link_start, mass 0.8; collision cylinder length=0.05 radius=0.025; visual cylinder length=0.06 radius=0.025
- added link lidar_link
- added link wrist_link_start, mass 0.8; collision cylinder length=0.05 radius=0.02; visual cylinder length=0.05 radius=0.02
- added link wrist_roll_link_cup, mass 0.1; collision cylinder length=0.02 radius=0.033; visual cylinder length=0.02 radius=0.033
- link base_link: mass 20.0 -> 40.0
- link elbow_link: geometry collision box size=0.04 0.04 0.3; visual box size=0.04 0.04 0.27
- link torso_link: mass 10.0 -> 2.0; geometry collision box size=0.3 0.3 0.5; visual box size=0.3 0.3 0.5
Joints:
- added joint elbow_joint_start: type fixed, parent shoulder_link, child elbow_link_start
- added joint lidar_joint: type fixed, parent torso_link, child lidar_link, origin xyz=0 0 0.18 rpy=0 0 0
- added joint wrist_joint_start: type fixed, parent wrist_pitch_link, child wrist_link_start
- added joint wrist_roll_joint_cup: type fixed, parent wrist_pitch_link, child wrist_roll_link_cup, origin xyz=0 0 0.03
- joint arm_base_joint: limit lower=-3.14 upper=0 effort=10.0 velocity=1.0 -> lower=-3.14 upper=3.14 effort=10.0 velocity=1.0
- joint bl_wheel_joint: axis 0 0 1 -> 0 0 -1
- joint br_wheel_joint: axis 0 0 1 -> 0 0 -1
- joint elbow_joint: limit lower=0.0 upper=2.0 effort=10.0 velocity=1.0 -> lower=-0.5 upper=2.0 effort=10.0 velocity=1.0
- joint fl_wheel_joint: axis 0 0 1 -> 0 0 -1
- joint fr_wheel_joint: axis 0 0 1 -> 0 0 -1
- joint lift_joint: axis 0 0 1 -> (none); limit lower=0.0 upper=0.3 effort=100.0 velocity=0.5 -> (none); origin xyz=0 -0.1 -0.15 rpy=0 0 0 -> xyz=0 0 0.22 rpy=0 0 0; type prismatic -> fixed
- joint shoulder_joint: limit lower=0.0 upper=1.57 effort=10.0 velocity=1.0 -> lower=-1.0 upper=1.57 effort=10.0 velocity=1.0
- joint torso_fixed_joint: origin xyz=0 0 0.25 -> xyz=0 0 0.3
- joint wrist_pitch_joint: origin xyz=0 0 0.3 -> xyz=0 0 0.29 rpy=0 0.4 0
- joint wrist_roll_joint: origin xyz=0 0 0.05 -> xyz=0 0 0.056

Commit message: debug: fix table pos so that I can work in peace

File: src/robot/robot.urdf (robot description, URDF)
Before this commit: robot iis_robot, 21 links, 20 joints
Links:
- link base_link: mass 5.0 -> 40.0
Joints:
- joint camera_joint: origin xyz=0.25 0 0.15 rpy=0 0 0 -> xyz=0.12 0 0.27 rpy=0 0.2 0; parent torso_link -> gripper_base
- joint lift_joint: axis (none) -> 0 0 1; limit (none) -> lower=0.0 upper=0.3 effort=100.0 velocity=0.5; type fixed -> prismatic
- joint wrist_pitch_joint: origin xyz=0 0 0.29 -> xyz=0 0 0.29 rpy=0 0.4 0

Commit message: fix: use robot.urdf from src/robot

File: src/robot/robot.urdf (robot description, URDF)
Before this commit: robot iis_robot, 21 links, 20 joints
Links:
- link base_link: mass 5.0 -> 40.0
Joints:
- joint camera_joint: origin xyz=0.25 0 0.15 rpy=0 0 0 -> xyz=0.12 0 0.27 rpy=0 0.2 0
- joint lift_joint: axis (none) -> 0 0 1; limit (none) -> lower=0.0 upper=0.3 effort=100.0 velocity=0.5; type fixed -> prismatic
- joint wrist_pitch_joint: origin xyz=0 0 0.29 -> xyz=0 0 0.29 rpy=0 0.4 0

Commit message: working on ik

File: src/robot/robot.urdf (robot description, URDF)
Before this commit: robot iis_robot, 21 links, 20 joints
Joints:
- joint camera_joint: origin xyz=0.12 0 0.27 rpy=0 0.2 0 -> xyz=0 0 0 rpy=0 0 0
- joint lidar_joint: origin xyz=0 0 0.18 rpy=0 0 0 -> xyz=0 0 0.35 rpy=0 0 0; parent torso_link -> base_link
- joint lift_joint: type prismatic -> fixed

Commit message: fixed grasping

File: src/robot/robot.urdf (robot description, URDF)
Before this commit: robot iis_robot, 21 links, 20 joints
Joints:
- joint camera_joint: origin xyz=0.12 0 0.27 rpy=0 0.2 0 -> xyz=0.22 0 0.27 rpy=0 0.2 0
- joint left_finger_joint: origin xyz=0.04 0.04 0 rpy=0 0 0 -> xyz=0.05 0.044 0 rpy=0 0 0
- joint right_finger_joint: origin xyz=0.04 -0.04 0 rpy=0 0 0 -> xyz=0.05 -0.044 0 rpy=0 0 0

Commit message: Fix gripper dimensions and grasp distance threshold

File: src/robot/robot.urdf (robot description, URDF)
Before this commit: robot iis_robot, 21 links, 20 joints
Links:
- link gripper_base: geometry collision box size=0.05 0.1 0.05; visual box size=0.05 0.15 0.05
- link left_finger: geometry collision box size=0.08 0.01 0.02; visual box size=0.08 0.01 0.05
- link right_finger: geometry collision box size=0.08 0.01 0.02; visual box size=0.08 0.01 0.05
Joints:
- joint left_finger_joint: origin xyz=0.05 0.044 0 rpy=0 0 0 -> xyz=0.05 0.07 0 rpy=0 0 0
- joint right_finger_joint: origin xyz=0.05 -0.044 0 rpy=0 0 0 -> xyz=0.05 -0.07 0 rpy=0 0 0
